Commit message: Update nannanananan.xacro

File: extract/nannanananan_description/urdf/nannanananan.xacro (robot description, xacro)
@@ -68,5 +68,5 @@
   <parent link="base_link"/>
   <child link="whell_2_1"/>
-  <axis xyz="-0.0 1.0 0.0"/>
+  <axis xyz="0.0 1.0 0.0"/>
 </joint>
 <joint name="Rev2" type="continuous">
@@ -74,5 +74,5 @@
   <parent link="base_link"/>
   <child link="whell_1"/>
-  <axis xyz="0.0 -1.0 -0.0"/>
+  <axis xyz="0.0 1.0 0.0"/>
 </joint>
 </robot>
